File: TA726.kicad_pcb (KiCad board)
At the start: 2 copper layers, 19.2 x 27.7 mm, 15 parts, among them J1 Conn_02x05_Counter_Clockwise, U1 MAT14ARZ, U2 OP97FSZ

Commit message: rotated trimmer
Parts:
- added REF**: DIP-10_W7.62mm, Package_DIP:DIP-10_W7.62mm, B.Cu at (211.2, 94.3)
- U1: value MAT14ARZ -> MAT14
- moved RV1 3.59 mm to (211.3, 79.3), turned to 0 degrees
- moved D1 2.08 mm to (218.0, 89.6)
- moved C12 1.49 mm to (204.9, 83.4)
- moved C13 1.49 mm to (217.7, 83.4)
- moved C2 1.20 mm to (217.2, 99.4)
- moved R1 0.91 mm to (210.4, 86.3)
- moved C3 0.84 mm to (213.5, 86.3)
Connections:
- net /BX renamed Net-(U1B-B)
- U1 pad 1: /C1 -> /C2
- U1 pad 12: /E2 -> /E1
- U1 pad 13: /B2 -> /B1
- U1 pad 14: /C2 -> /C1
- U1 pad 2: /B1 -> /B2
- U1 pad 3: /E1 -> /E2
Routing:
- net /E1: track 19.1 -> 4.05 mm
- net /E2: track 23.7 -> 11.9 mm
- net /B1: track 17.7 -> 7.68 mm
- net /C1: track 5.19 -> 9.37 mm
- net /C2: track 8.72 -> 5.08 mm
- net Net-(R1-Pad1): track 5.73 -> 9.17 mm
- net Net-(U2--): track 17.5 -> 14.9 mm
- net VCC: track 46.8 -> 44.4 mm
- net Net-(D1-K): track 13.9 -> 12.1 mm
- net Net-(D1-A): track 6.44 -> 4.71 mm
- net VEE: track 29.1 -> 30.2 mm
- net Net-(U1B-B): track 28.3 -> 27.3 mm
- net /B2: track 8.49 -> 9.50 mm
- net GND: track 7.95 -> 7.11 mm
