File: TA726.kicad_sch (KiCad schematic)
At the start: 15 parts, among them J1 Conn_02x05_Counter_Clockwise, U1 MAT14ARZ, U2 OP97FSZ

Commit message: rotated trimmer
Parts:
- removed U1: MAT14ARZ, Triglav_Modular:SO-14_3.9x8.65mm_P1.27mm, symbol Triglav_Modular:MAT14ARZ
- added U1: MAT14, Triglav_Modular:SO-14_3.9x8.65mm_P1.27mm, symbol Triglav_Modular:MAT14
Connections:
- net B1: now also U1.13 (B)
- net B2: now also U1.2 (B)
- net C1: now also U1.14 (C)
- net C2: now also U1.1 (C)
- net E1: now also U1.12 (E)
- net E2: now also U1.3 (E)
- net GND: now also U1.5 (E)
- net V-: now also U1.4 (Substrate)
- net VCC: now also U1.8 (C)
- net VEE: now also U1.11 (Substrate)
- net at R2.2, R5.2: now also U1.9 (B)
- net at R3.1: now also U1.10 (E)
- net BX: no longer names the net of C1.1, R4.2, U2.3 (+)
- net BX: now also U1.6 (B), U1.7 (C)
